File: Kicad-Midi2CV.sch (KiCad schematic (older format))
At the start: 9 parts, among them U2 EL814

Commit message: GND and LED
GND added
MIDI CH LED indicators added
Parts:
- added D? (x4): LED, LED_THT:LED_D3.0mm_Horizontal_O6.35mm_Z6.0mm, symbol Device:LED
- added R? (x2): R, symbol Device:R
- added R? (x5): 680R, Resistor_SMD:R_0805_2012Metric_Pad1.15x1.40mm_HandSolder, symbol Device:R
Connections:
- net labels added: GND
- wire segments 24 -> 64

Commit message: I2C
Power and pullup
Parts:
- removed R? (x4): R, symbol Device:R
- added J?: Conn_01x04, symbol Connector_Generic:Conn_01x04
- added R? (x2): 1k, Resistor_SMD:R_0805_2012Metric_Pad1.15x1.40mm_HandSolder, symbol Device:R
- added R? (x2): 8k2, Resistor_SMD:R_0805_2012Metric_Pad1.15x1.40mm_HandSolder, symbol Device:R
Connections:
- wire segments 64 -> 105

Commit message: reorganize
boxes around functions
Parts:
- added C?: C, symbol Device:C
- added C?: CP, symbol Device:CP
- added J?: Barrel_Jack, symbol Connector:Barrel_Jack
Connections:
- wire segments 105 -> 111

Commit message: MIDI pinout
correct
Parts:
- R?: value 680R -> 220R
Connections:
- wire segments 111 -> 109
Changed lines of the file:
@@
 L Connector:DIN-5 J?
 U 1 1 5C1C0BCC
-P 1300 2750
-F 0 "J?" H 1300 2476 50  0000 C CNN
-F 1 "DIN-5" H 1300 2385 50  0000 C CNN
-F 2 "" H 1300 2750 50  0001 C CNN
-F 3 "http://www.mouser.com/ds/2/18/40_c091_abd_e-75918.pdf" H 1300 2750 50  0001 C CNN
-	1    1300 2750
+P 1250 2500
+F 0 "J?" H 1250 2226 50  0000 C CNN
+F 1 "DIN-5" H 1250 2135 50  0000 C CNN
+F 2 "" H 1250 2500 50  0001 C CNN
+F 3 "http://www.mouser.com/ds/2/18/40_c091_abd_e-75918.pdf" H 1250 2500 50  0001 C CNN
+	1    1250 2500
 	1    0    0    -1
 $EndComp
@@
 	2550 2400 2800 2400
 Wire Wire Line
-	1950 2600 1600 2600
-Wire Wire Line
-	1600 2600 1600 2650
-Wire Wire Line
-	1000 2400 1000 2650
-Wire Wire Line
 	6000 3300 5600 3300
 Wire Wire Line
@@
 L Device:R R?
 U 1 1 5C1CFCF0
-P 1700 2400
-F 0 "R?" V 1493 2400 50  0000 C CNN
-F 1 "680R" V 1584 2400 50  0000 C CNN
-F 2 "Resistor_SMD:R_0805_2012Metric_Pad1.15x1.40mm_HandSolder" V 1630 2400 50  0001 C CNN
-F 3 "~" H 1700 2400 50  0001 C CNN
-	1    1700 2400
+P 1750 2400
+F 0 "R?" V 1543 2400 50  0000 C CNN
+F 1 "220R" V 1634 2400 50  0000 C CNN
+F 2 "Resistor_SMD:R_0805_2012Metric_Pad1.15x1.40mm_HandSolder" V 1680 2400 50  0001 C CNN
+F 3 "~" H 1750 2400 50  0001 C CNN
+	1    1750 2400
 	0    1    1    0
 $EndComp
-Wire Wire Line
-	1850 2400 1950 2400
-Wire Wire Line
-	1000 2400 1550 2400
 Wire Wire Line
 	3200 3850 3000 3850
@@
 Wire Notes Line
 	850  5850 850  3400
+Wire Wire Line
+	1900 2400 1950 2400
+Wire Wire Line
+	1550 2600 1950 2600
+Wire Wire Line
+	1550 2400 1600 2400
 $EndSCHEMATC

Commit message: DIN-5 footprint
added from http://smisioto.no-ip.org/elettronica/kicad/kicad-en.htm
Parts:
- J?: footprint (none) -> w_conn_av:din-5
Changed lines of the file:
@@
 F 0 "J?" H 1250 2226 50  0000 C CNN
 F 1 "DIN-5" H 1250 2135 50  0000 C CNN
-F 2 "" H 1250 2500 50  0001 C CNN
+F 2 "w_conn_av:din-5" H 1250 2500 50  0001 C CNN
 F 3 "http://www.mouser.com/ds/2/18/40_c091_abd_e-75918.pdf" H 1250 2500 50  0001 C CNN
 	1    1250 2500

Commit message: Channel select
Rotary encoder added for MIDI channel select
Parts:
- added SW?: Rotary_Encoder_Switch, symbol Device:Rotary_Encoder_Switch
Connections:
- wire segments 109 -> 115
Changed lines of the file:
@@
 Wire Wire Line
 	1550 2400 1600 2400
+$Comp
+L Device:Rotary_Encoder_Switch SW?
+U 1 1 5C253AC2
+P 3200 5300
+F 0 "SW?" H 3200 4933 50  0000 C CNN
+F 1 "Rotary_Encoder_Switch" H 3200 5024 50  0000 C CNN
+F 2 "" H 3050 5460 50  0001 C CNN
+F 3 "~" H 3200 5560 50  0001 C CNN
+	1    3200 5300
+	-1   0    0    1
+$EndComp
+Wire Wire Line
+	3500 5200 4200 5200
+Wire Wire Line
+	4200 5200 4200 3200
+Wire Wire Line
+	4200 3200 4600 3200
+Wire Wire Line
+	4600 3300 4300 3300
+Wire Wire Line
+	4300 3300 4300 5400
+Wire Wire Line
+	3500 5400 4300 5400
 $EndSCHEMATC

Commit message: Footprints
Cap, BJT, Conn, Etc
Parts:
- C1: renamed from C?; footprint (none) -> Capacitor_THT:CP_Radial_D5.0mm_P2.50mm
- C2: renamed from C?; footprint (none) -> Capacitor_SMD:C_0805_2012Metric_Pad1.15x1.40mm_HandSolder
- IC1, IC2: renamed from IC?; footprint (none) -> Connector_PinSocket_2.54mm:PinSocket_1x06_P2.54mm_Vertical
- J1: renamed from J?; footprint (none) -> Connector_BarrelJack:BarrelJack_CUI_PJ-063AH_Horizontal
- Q1: renamed from Q?; footprint SOT23 -> Package_TO_SOT_SMD:SOT-23_Handsoldering
- U2: footprint (none) -> OptoDevice:Panasonic_APV-AQY_SSOP-4_4.45x2.65mm_P1.27mm
- gave numbers to parts that had none: 17
Changed lines of the file:
@@
 F 0 "U2" H 2250 2825 50  0000 C CNN
 F 1 "EL814" H 2250 2734 50  0000 C CNN
-F 2 "" H 2050 2300 50  0001 L CIN
+F 2 "OptoDevice:Panasonic_APV-AQY_SSOP-4_4.45x2.65mm_P1.27mm" H 2050 2300 50  0001 L CIN
 F 3 "http://www.everlight.com/file/ProductFile/EL814.pdf" H 2275 2500 50  0001 L CNN
 	1    2250 2500
@@
 $EndComp
 $Comp
-L MMBT2222A:MMBT2222A Q?
+L MMBT2222A:MMBT2222A Q1
 U 1 1 5C1C0AF7
 P 3000 2600
-F 0 "Q?" H 3141 2646 50  0000 L CNN
+F 0 "Q1" H 3141 2646 50  0000 L CNN
 F 1 "MMBT2222A" H 3141 2555 50  0000 L CNN
-F 2 "SOT23" H 3000 2600 50  0001 L BNN
+F 2 "Package_TO_SOT_SMD:SOT-23_Handsoldering" H 3000 2600 50  0001 L BNN
 F 3 "Unavailable" H 3000 2600 50  0001 L BNN
 F 4 "None" H 3000 2600 50  0001 L BNN "Field4"
 F 5 "ON" H 3000 2600 50  0001 L BNN "Field5"
-F 6 "" H 3000 2600 50  0001 L BNN "Field6"
-F 7 "MMBT2222A" H 3000 2600 50  0001 L BNN "Field7"
-F 8 "TO-236-3 Taitron" H 3000 2600 50  0001 L BNN "Field8"
+F 6 "MMBT2222A" H 3000 2600 50  0001 L BNN "Field7"
+F 7 "TO-236-3 Taitron" H 3000 2600 50  0001 L BNN "Field8"
 	1    3000 2600
 	1    0    0    -1
 $EndComp
 $Comp
-L Connector:DIN-5 J?
+L Connector:DIN-5 J3
 U 1 1 5C1C0BCC
 P 1250 2500
-F 0 "J?" H 1250 2226 50  0000 C CNN
+F 0 "J3" H 1250 2226 50  0000 C CNN
 F 1 "DIN-5" H 1250 2135 50  0000 C CNN
 F 2 "w_conn_av:din-5" H 1250 2500 50  0001 C CNN
@@
 $EndComp
 $Comp
-L Analog_DAC:MCP4728 U?
+L Analog_DAC:MCP4728 U1
 U 1 1 5C1C0F59
 P 7200 4800
-F 0 "U?" H 7200 5278 50  0000 C CNN
+F 0 "U1" H 7200 5278 50  0000 C CNN
 F 1 "MCP4728" H 7200 5187 50  0000 C CNN
 F 2 "Package_SO:MSOP-10_3x3mm_P0.5mm" H 7200 4200 50  0001 C CNN
@@
 $EndComp
 $Comp
-L aj_adc_dac:MCP4725module IC?
+L aj_adc_dac:MCP4725module IC2
 U 1 1 5C1C16C6
 P 7200 3400
-F 0 "IC?" H 7991 3453 60  0000 L CNN
+F 0 "IC2" H 7991 3453 60  0000 L CNN
 F 1 "MCP4725module" H 7991 3347 60  0000 L CNN
-F 2 "" H 7200 3400 50  0001 C CNN
+F 2 "Connector_PinSocket_2.54mm:PinSocket_1x06_P2.54mm_Vertical" H 7200 3400 50  0001 C CNN
 F 3 "" H 7200 3400 50  0001 C CNN
 	1    7200 3400
@@
 	7825 3300 7750 3300
 $Comp
-L aj_adc_dac:MCP4725module IC?
+L aj_adc_dac:MCP4725module IC1
 U 1 1 5C1C326B
 P 7200 2350
-F 0 "IC?" H 7991 2403 60  0000 L CNN
+F 0 "IC1" H 7991 2403 60  0000 L CNN
 F 1 "MCP4725module" H 7991 2297 60  0000 L CNN
-F 2 "" H 7200 2350 50  0001 C CNN
+F 2 "Connector_PinSocket_2.54mm:PinSocket_1x06_P2.54mm_Vertical" H 7200 2350 50  0001 C CNN
 F 3 "" H 7200 2350 50  0001 C CNN
 	1    7200 2350
@@
 	4500 3400 4600 3400
 $Comp
-L Device:LED D?
+L Device:LED D1
 U 1 1 5C1CEEC6
 P 2400 3850
-F 0 "D?" H 2391 4066 50  0000 C CNN
+F 0 "D1" H 2391 4066 50  0000 C CNN
 F 1 "LED" H 2391 3975 50  0000 C CNN
 F 2 "LED_THT:LED_D3.0mm_Horizontal_O6.35mm_Z6.0mm" H 2400 3850 50  0001 C CNN
@@
 $EndComp
 $Comp
-L Device:LED D?
+L Device:LED D2
 U 1 1 5C1CEF6A
 P 2400 4150
-F 0 "D?" H 2391 4366 50  0000 C CNN
+F 0 "D2" H 2391 4366 50  0000 C CNN
 F 1 "LED" H 2391 4275 50  0000 C CNN
 F 2 "LED_THT:LED_D3.0mm_Horizontal_O6.35mm_Z6.0mm" H 2400 4150 50  0001 C CNN
@@
 $EndComp
 $Comp
-L Device:LED D?
+L Device:LED D3
 U 1 1 5C1CF002
 P 2400 4500
-F 0 "D?" H 2391 4716 50  0000 C CNN
+F 0 "D3" H 2391 4716 50  0000 C CNN
 F 1 "LED" H 2391 4625 50  0000 C CNN
 F 2 "LED_THT:LED_D3.0mm_Horizontal_O6.35mm_Z6.0mm" H 2400 4500 50  0001 C CNN
@@
 $EndComp
 $Comp
-L Device:LED D?
+L Device:LED D4
 U 1 1 5C1CF008
 P 2400 4800
-F 0 "D?" H 2391 5016 50  0000 C CNN
+F 0 "D4" H 2391 5016 50  0000 C CNN
 F 1 "LED" H 2391 4925 50  0000 C CNN
 F 2 "LED_THT:LED_D3.0mm_Horizontal_O6.35mm_Z6.0mm" H 2400 4800 50  0001 C CNN
@@
 $EndComp
 $Comp
-L Device:R R?
+L Device:R R6
 U 1 1 5C1CFAFB
 P 2850 3850
-F 0 "R?" V 2643 3850 50  0000 C CNN
+F 0 "R6" V 2643 3850 50  0000 C CNN
 F 1 "680R" V 2734 3850 50  0000 C CNN
 F 2 "Resistor_SMD:R_0805_2012Metric_Pad1.15x1.40mm_HandSolder" V 2780 3850 50  0001 C CNN
@@
 $EndComp
 $Comp
-L Device:R R?
+L Device:R R7
 U 1 1 5C1CFC0E
 P 2850 4150
-F 0 "R?" V 2643 4150 50  0000 C CNN
+F 0 "R7" V 2643 4150 50  0000 C CNN
 F 1 "680R" V 2734 4150 50  0000 C CNN
 F 2 "Resistor_SMD:R_0805_2012Metric_Pad1.15x1.40mm_HandSolder" V 2780 4150 50  0001 C CNN
@@
 $EndComp
 $Comp
-L Device:R R?
+L Device:R R8
 U 1 1 5C1CFC52
 P 2850 4500
-F 0 "R?" V 2643 4500 50  0000 C CNN
+F 0 "R8" V 2643 4500 50  0000 C CNN
 F 1 "680R" V 2734 4500 50  0000 C CNN
 F 2 "Resistor_SMD:R_0805_2012Metric_Pad1.15x1.40mm_HandSolder" V 2780 4500 50  0001 C CNN
@@
 $EndComp
 $Comp
-L Device:R R?
+L Device:R R9
 U 1 1 5C1CFCA2
 P 2850 4800
-F 0 "R?" V 2643 4800 50  0000 C CNN
+F 0 "R9" V 2643 4800 50  0000 C CNN
 F 1 "680R" V 2734 4800 50  0000 C CNN
 F 2 "Resistor_SMD:R_0805_2012Metric_Pad1.15x1.40mm_HandSolder" V 2780 4800 50  0001 C CNN
@@
 $EndComp
 $Comp
-L Device:R R?
+L Device:R R4
 U 1 1 5C1CFCF0
 P 1750 2400
-F 0 "R?" V 1543 2400 50  0000 C CNN
+F 0 "R4" V 1543 2400 50  0000 C CNN
 F 1 "220R" V 1634 2400 50  0000 C CNN
 F 2 "Resistor_SMD:R_0805_2012Metric_Pad1.15x1.40mm_HandSolder" V 1680 2400 50  0001 C CNN
@@
 	2700 4800 2550 4800
 $Comp
-L power:GND #PWR?
+L power:GND #PWR05
 U 1 1 5C1D9D12
 P 2050 4950
-F 0 "#PWR?" H 2050 4700 50  0001 C CNN
+F 0 "#PWR05" H 2050 4700 50  0001 C CNN
 F 1 "GND" H 2055 4777 50  0000 C CNN
 F 2 "" H 2050 4950 50  0001 C CNN
@@
 $EndComp
 $Comp
-L power:GND #PWR?
+L power:GND #PWR06
 U 1 1 5C1D9DC0
 P 7200 5300
-F 0 "#PWR?" H 7200 5050 50  0001 C CNN
+F 0 "#PWR06" H 7200 5050 50  0001 C CNN
 F 1 "GND" H 7205 5127 50  0000 C CNN
 F 2 "" H 7200 5300 50  0001 C CNN
@@
 $EndComp
 $Comp
-L power:GND #PWR?
+L power:GND #PWR03
 U 1 1 5C1D9DFA
 P 7200 3850
-F 0 "#PWR?" H 7200 3600 50  0001 C CNN
+F 0 "#PWR03" H 7200 3600 50  0001 C CNN
 F 1 "GND" H 7205 3677 50  0000 C CNN
 F 2 "" H 7200 3850 50  0001 C CNN
@@
 $EndComp
 $Comp
-L power:GND #PWR?
+L power:GND #PWR02
 U 1 1 5C1D9E7D
 P 7200 2800
-F 0 "#PWR?" H 7200 2550 50  0001 C CNN
+F 0 "#PWR02" H 7200 2550 50  0001 C CNN
 F 1 "GND" H 7205 2627 50  0000 C CNN
 F 2 "" H 7200 2800 50  0001 C CNN
@@
 $EndComp
 $Comp
-L power:GND #PWR?
+L power:GND #PWR04
 U 1 1 5C1D9F00
 P 5150 4050
-F 0 "#PWR?" H 5150 3800 50  0001 C CNN
+F 0 "#PWR04" H 5150 3800 50  0001 C CNN
 F 1 "GND" H 5155 3877 50  0000 C CNN
 F 2 "" H 5150 4050 50  0001 C CNN
@@
 	2050 4800 2050 4950
 $Comp
-L Device:R R?
+L Device:R R3
 U 1 1 5C1DFF32
 P 3100 2100
-F 0 "R?" H 3030 2054 50  0000 R CNN
+F 0 "R3" H 3030 2054 50  0000 R CNN
 F 1 "1k" H 3030 2145 50  0000 R CNN
 F 2 "Resistor_SMD:R_0805_2012Metric_Pad1.15x1.40mm_HandSolder" V 3030 2100 50  0001 C CNN
@@
 	3100 1950 3100 1850
 $Comp
-L Device:R R?
+L Device:R R5
 U 1 1 5C1E3615
 P 2750 2850
-F 0 "R?" H 2680 2804 50  0000 R CNN
+F 0 "R5" H 2680 2804 50  0000 R CNN
 F 1 "1k" H 2680 2895 50  0000 R CNN
 F 2 "Resistor_SMD:R_0805_2012Metric_Pad1.15x1.40mm_HandSolder" V 2680 2850 50  0001 C CNN
@@
 Connection ~ 2050 3850
 $Comp
-L Device:R R?
+L Device:R R1
 U 1 1 5C1E9F2A
 P 6350 1850
-F 0 "R?" H 6280 1804 50  0000 R CNN
+F 0 "R1" H 6280 1804 50  0000 R CNN
 F 1 "8k2" H 6280 1895 50  0000 R CNN
 F 2 "Resistor_SMD:R_0805_2012Metric_Pad1.15x1.40mm_HandSolder" V 6280 1850 50  0001 C CNN
@@
 $EndComp
 $Comp
-L Device:R R?
+L Device:R R2
 U 1 1 5C1E9FAC
 P 6450 1850
-F 0 "R?" H 6380 1804 50  0000 R CNN
+F 0 "R2" H 6380 1804 50  0000 R CNN
 F 1 "8k2" H 6380 1895 50  0000 R CNN
 F 2 "Resistor_SMD:R_0805_2012Metric_Pad1.15x1.40mm_HandSolder" V 6380 1850 50  0001 C CNN
@@
 Connection ~ 7900 2000
 $Comp
-L Connector_Generic:Conn_01x04 J?
+L Connector_Generic:Conn_01x04 J2
 U 1 1 5C21A17B
 P 6000 1800
-F 0 "J?" H 6080 1792 50  0000 L CNN
+F 0 "J2" H 6080 1792 50  0000 L CNN
 F 1 "Conn_01x04" H 6080 1701 50  0000 L CNN
 F 2 "" H 6000 1800 50  0001 C CNN
@@
 	5200 1750 5200 1800
 $Comp
-L power:GND #PWR?
+L power:GND #PWR01
 U 1 1 5C2240E9
 P 5800 2050
-F 0 "#PWR?" H 5800 1800 50  0001 C CNN
+F 0 "#PWR01" H 5800 1800 50  0001 C CNN
 F 1 "GND" H 5805 1877 50  0000 C CNN
 F 2 "" H 5800 2050 50  0001 C CNN
@@
 Connection ~ 6350 1650
 $Comp
-L Device:C C?
+L Device:C C2
 U 1 1 5C22F1AA
 P 2500 1100
-F 0 "C?" H 2615 1146 50  0000 L CNN
+F 0 "C2" H 2615 1146 50  0000 L CNN
 F 1 "C" H 2615 1055 50  0000 L CNN
-F 2 "" H 2538 950 50  0001 C CNN
+F 2 "Capacitor_SMD:C_0805_2012Metric_Pad1.15x1.40mm_HandSolder" H 2538 950 50  0001 C CNN
 F 3 "~" H 2500 1100 50  0001 C CNN
 	1    2500 1100
@@
 $EndComp
 $Comp
-L Device:CP C?
+L Device:CP C1
 U 1 1 5C22F286
 P 2100 1100
-F 0 "C?" H 2218 1146 50  0000 L CNN
+F 0 "C1" H 2218 1146 50  0000 L CNN
 F 1 "CP" H 2218 1055 50  0000 L CNN
-F 2 "" H 2138 950 50  0001 C CNN
+F 2 "Capacitor_THT:CP_Radial_D5.0mm_P2.50mm" H 2138 950 50  0001 C CNN
 F 3 "~" H 2100 1100 50  0001 C CNN
 	1    2100 1100
@@
 $EndComp
 $Comp
-L Connector:Barrel_Jack J?
+L Connector:Barrel_Jack J1
 U 1 1 5C22F3A0
 P 1250 1100
-F 0 "J?" H 1305 1425 50  0000 C CNN
+F 0 "J1" H 1305 1425 50  0000 C CNN
 F 1 "Barrel_Jack" H 1305 1334 50  0000 C CNN
-F 2 "" H 1300 1060 50  0001 C CNN
+F 2 "Connector_BarrelJack:BarrelJack_CUI_PJ-063AH_Horizontal" H 1300 1060 50  0001 C CNN
 F 3 "~" H 1300 1060 50  0001 C CNN
 	1    1250 1100
@@
 	1550 2400 1600 2400
 $Comp
-L Device:Rotary_Encoder_Switch SW?
+L Device:Rotary_Encoder_Switch SW1
 U 1 1 5C253AC2
 P 3200 5300
-F 0 "SW?" H 3200 4933 50  0000 C CNN
+F 0 "SW1" H 3200 4933 50  0000 C CNN
 F 1 "Rotary_Encoder_Switch" H 3200 5024 50  0000 C CNN
 F 2 "" H 3050 5460 50  0001 C CNN

Commit message: Footprints
footprint PL814
Parts:
- U2: footprint OptoDevice:Panasonic_APV-AQY_SSOP-4_4.45x2.65mm_P1.27mm -> Package_DIP:DIP-4_W7.62mm_LongPads
Changed lines of the file:
@@
 F 0 "U2" H 2250 2825 50  0000 C CNN
 F 1 "EL814" H 2250 2734 50  0000 C CNN
-F 2 "OptoDevice:Panasonic_APV-AQY_SSOP-4_4.45x2.65mm_P1.27mm" H 2050 2300 50  0001 L CIN
+F 2 "Package_DIP:DIP-4_W7.62mm_LongPads" H 2050 2300 50  0001 L CIN
 F 3 "http://www.everlight.com/file/ProductFile/EL814.pdf" H 2275 2500 50  0001 L CNN
 	1    2250 2500
