File: Kicad-Midi2CV.sch (KiCad schematic (older format))
At the start: 29 parts, among them IC1 MCP4725module, IC2 MCP4725module, J1 Barrel_Jack, J2 Conn_01x04, J3 DIN-5, Q1 MMBT2222A, SW1 Rotary_Encoder_Switch, U1 EL814, U2 MCP4728

Commit message: Power redraw
Redraw power
Parts:
- added C? (x2): C, Capacitor_SMD:C_0805_2012Metric_Pad1.15x1.40mm_HandSolder, symbol Device:C
- added R?: 680R, Resistor_SMD:R_0805_2012Metric_Pad1.15x1.40mm_HandSolder, symbol Device:R
Other:
- moved on the sheet: A1, C1, C2, C?, D1, D2, D3, D4, J1, J2, J3, Q1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

Commit message: Jack
PJ398SM x2 jack
Parts:
- added J? (x2): AudioJack2_Ground_Switch, Connector_Audio:Jack_3.5mm_QingPu_WQP-PJ398SM_Vertical_CircularHoles, symbol Connector:AudioJack2_Ground_Switch
Changed lines of the file:
@@
 Wire Wire Line
 	5150 2850 5550 2850
+$Comp
+L Connector:AudioJack2_Ground_Switch J?
+U 1 1 5C2C7CBB
+P 10200 2900
+F 0 "J?" H 9967 2971 50  0000 R CNN
+F 1 "AudioJack2_Ground_Switch" H 9967 2880 50  0000 R CNN
+F 2 "Connector_Audio:Jack_3.5mm_QingPu_WQP-PJ398SM_Vertical_CircularHoles" H 10200 2900 50  0001 C CNN
+F 3 "~" H 10200 2900 50  0001 C CNN
+	1    10200 2900
+	-1   0    0    -1
+$EndComp
+$Comp
+L Connector:AudioJack2_Ground_Switch J?
+U 1 1 5C2C7E1B
+P 10200 3350
+F 0 "J?" H 9967 3421 50  0000 R CNN
+F 1 "AudioJack2_Ground_Switch" H 9967 3330 50  0000 R CNN
+F 2 "Connector_Audio:Jack_3.5mm_QingPu_WQP-PJ398SM_Vertical_CircularHoles" H 10200 3350 50  0001 C CNN
+F 3 "~" H 10200 3350 50  0001 C CNN
+	1    10200 3350
+	-1   0    0    -1
+$EndComp
 $EndSCHEMATC

Commit message: LED tag
Labels for LED, button, encoder and Gates
Parts:
- added D?: LED, LED_THT:LED_D3.0mm_Horizontal_O6.35mm_Z6.0mm, symbol Device:LED
- added R?: 680R, Resistor_SMD:R_0805_2012Metric_Pad1.15x1.40mm_HandSolder, symbol Device:R
- R?: value 680R -> 10M
Connections:
- net labels added: Btn, Gate1, Gate2, LED-sel, LED1, LED2, LED3, LED4
- wire segments 131 -> 139
Other:
- moved on the sheet: D1, D2, D3, D4, R6, R7, R8, R9

Commit message: Multi IO
Gate3/4
Encoder to A0, A1, A2
A3 as input
LED sel2
Parts:
- added C?: 10n, Capacitor_SMD:C_0805_2012Metric_Pad1.15x1.40mm_HandSolder, symbol Device:C
- added D?: LED, LED_THT:LED_D3.0mm_Horizontal_O6.35mm_Z6.0mm, symbol Device:LED
- added R?: 10k, Resistor_SMD:R_0805_2012Metric_Pad1.15x1.40mm_HandSolder, symbol Device:R
- added R?: 680R, Resistor_SMD:R_0805_2012Metric_Pad1.15x1.40mm_HandSolder, symbol Device:R
Connections:
- net labels added: A1, A2, A3, CV1, CV2, CV3, CV4, Gate3, Gate4, LDAC, LED-sel2, RDY-BSY, RX, SCL, SDA
- wire segments 139 -> 160
Other:
- moved on the sheet: A1, C?, D?, R3, R?

Commit message: Rev A ------- before check
9 Jacks attached
Slight rearrange
Parts:
- added J? (x7): AudioJack2_Ground_Switch, Connector_Audio:Jack_3.5mm_QingPu_WQP-PJ398SM_Vertical_CircularHoles, symbol Connector:AudioJack2_Ground_Switch
- gave numbers to parts that had none: 15
- renumbered J3 to J5, R9 to R10, R1 to R2, R2 to R3, R3 to R4, R4 to R5, R5 to R6, R6 to R7, R7 to R8, R8 to R9
Connections:
- wire segments 160 -> 200
Other:
- moved on the sheet: C5, C6, C7, R13, R14, R15

Commit message: Rev A2 -  prior to footprint
CV1 and CV2 with gain adjustment
Parts:
- added J2: DIN-5, w_conn_av:din-5, symbol Connector:DIN-5
- added R2: 220R, Resistor_SMD:R_0805_2012Metric_Pad1.15x1.40mm_HandSolder, symbol Device:R
- added R6, R9: 0R, Resistor_SMD:R_0805_2012Metric_Pad1.15x1.40mm_HandSolder, symbol Device:R
- added R? (x4): 10k, Resistor_SMD:R_0805_2012Metric_Pad1.15x1.40mm_HandSolder, symbol Device:R
- added RV? (x2): 10k, symbol Device:R_POT
- added U? (x2): TL072, symbol Amplifier_Operational:TL072
- gave numbers to parts that had none: 7
- renumbered J2 to J4, J3 to J5, J4 to J6, J5 to J8, R7 to R10, R8 to R11, R9 to R12, R10 to R13, R11 to R14, R12 to R15, R13 to R16, R14 to R17, R15 to R18, R2 to R3, R3 to R4, R4 to R5, R5 to R7, R6 to R8
Connections:
- net labels added: CV1Gain, CV2Gain
- wire segments 200 -> 234
Other:
- note added: "Encoder Control"
- note added: "I2C DAC"
- note added: "LED Signals"
- note added: "MIDI IN"

Commit message: MIDI Out
Misc Cleanup
Parts:
- added Q1: MMBT2222A, Package_TO_SOT_SMD:SOT-23_Handsoldering, symbol MMBT2222A:MMBT2222A
- added R6, R8: 1k, Resistor_SMD:R_0805_2012Metric_Pad1.15x1.40mm_HandSolder, symbol Device:R
- J3: Function (none) -> VC input
- J5: Function (none) -> CV1 Out
- J6: Function (none) -> CV2 out
- gave numbers to parts that had none: 7
- renumbered J8 to J7, J7 to J8, Q1 to Q2, R4 to R10, R5 to R11, R7 to R12, R8 to R13, R6 to R14, R9 to R15, R10 to R16, R11 to R17, R12 to R18, R13 to R19, R14 to R20, R15 to R21, R16 to R22, R17 to R23, R18 to R24, R1 to R3, R2 to R7, R3 to R9, U1 to U2, U2 to U3
Connections:
- net labels added: MIDI-IN, MIDI-OUT, TX
- wire segments 234 -> 247
Other:
- moved on the sheet: J2, J7, Q2, R12, R13, R7, U2

Commit message: Footprints
Rotary encoder should be replaced...
Parts:
- RV1, RV2: footprint (none) -> Potentiometer_THT:Potentiometer_Alps_RK097_Single_Horizontal
- SW1: footprint (none) -> Rotary_Encoder:RotaryEncoder_Alps_EC11E-Switch_Vertical_H20mm
- U1: footprint (none) -> Package_SO:SO-8_5.3x6.2mm_P1.27mm
Changed lines of the file:
@@
-	1    0    0    -1
-$EndComp
-$Comp
-L power:GND #PWR015
-U 1 1 5C1D9F00
-P 4600 5450
-F 0 "#PWR015" H 4600 5200 50  0001 C CNN
-F 1 "GND" H 4605 5277 50  0000 C CNN
-F 2 "" H 4600 5450 50  0001 C CNN
-F 3 "" H 4600 5450 50  0001 C CNN
-	1    4600 5450
 	1    0    0    -1
 $EndComp
@@
 $EndComp
 Wire Wire Line
-	4600 5450 4600 5200
-Wire Wire Line
-	4600 5200 4650 5200
-Wire Wire Line
-	4550 5200 4600 5200
-Connection ~ 4600 5200
-Wire Wire Line
 	6400 3200 6100 3200
 Wire Wire Line
@@
 F 0 "SW1" H 2600 6783 50  0000 C CNN
 F 1 "Rotary_Encoder_Switch" H 2600 6874 50  0000 C CNN
-F 2 "" H 2450 7310 50  0001 C CNN
+F 2 "Rotary_Encoder:RotaryEncoder_Alps_EC11E-Switch_Vertical_H20mm" H 2450 7310 50  0001 C CNN
 F 3 "~" H 2600 7410 50  0001 C CNN
 	1    2600 7150
@@
 F 0 "U1" H 6650 1667 50  0000 C CNN
 F 1 "TL072" H 6650 1576 50  0000 C CNN
-F 2 "" H 6650 1300 50  0001 C CNN
+F 2 "Package_SO:SO-8_5.3x6.2mm_P1.27mm" H 6650 1300 50  0001 C CNN
 F 3 "http://www.ti.com/lit/ds/symlink/tl071.pdf" H 6650 1300 50  0001 C CNN
 	1    6650 1300
@@
 F 0 "U1" H 9850 1667 50  0000 C CNN
 F 1 "TL072" H 9850 1576 50  0000 C CNN
-F 2 "" H 9850 1300 50  0001 C CNN
+F 2 "Package_SO:SO-8_5.3x6.2mm_P1.27mm" H 9850 1300 50  0001 C CNN
 F 3 "http://www.ti.com/lit/ds/symlink/tl071.pdf" H 9850 1300 50  0001 C CNN
 	2    9850 1300
@@
 F 0 "RV1" H 7030 1046 50  0000 R CNN
 F 1 "10k" H 7030 955 50  0000 R CNN
-F 2 "" H 7100 1000 50  0001 C CNN
+F 2 "Potentiometer_THT:Potentiometer_Alps_RK097_Single_Horizontal" H 7100 1000 50  0001 C CNN
 F 3 "~" H 7100 1000 50  0001 C CNN
 	1    7100 1000
@@
 F 0 "RV2" H 10230 1046 50  0000 R CNN
 F 1 "10k" H 10230 955 50  0000 R CNN
-F 2 "" H 10300 1000 50  0001 C CNN
+F 2 "Potentiometer_THT:Potentiometer_Alps_RK097_Single_Horizontal" H 10300 1000 50  0001 C CNN
 F 3 "~" H 10300 1000 50  0001 C CNN
 	1    10300 1000
@@
 Wire Wire Line
 	2850 3600 2850 3650
+Wire Wire Line
+	4550 5200 4600 5200
+$Comp
+L power:GND #PWR0101
+U 1 1 5C912A2F
+P 4600 5300
+F 0 "#PWR0101" H 4600 5050 50  0001 C CNN
+F 1 "GND" H 4605 5127 50  0000 C CNN
+F 2 "" H 4600 5300 50  0001 C CNN
+F 3 "" H 4600 5300 50  0001 C CNN
+	1    4600 5300
+	1    0    0    -1
+$EndComp
+Wire Wire Line
+	4600 5300 4600 5200
+Connection ~ 4600 5200
+Wire Wire Line
+	4600 5200 4650 5200
 $EndSCHEMATC
