File: Kicad-Midi2CV.sch (KiCad schematic (older format))
At the start: 61 parts, among them IC1 MCP4725module, IC2 MCP4725module, J1 Barrel_Jack, J10 AudioJack2_Ground_Switch, J11 AudioJack2_Ground_Switch, J12 AudioJack2_Ground_Switch, J13 AudioJack2_Ground_Switch, J2 DIN-5, J3 AudioJack2_Ground_Switch, J4 Conn_01x04, J5 AudioJack2_Ground_Switch, J6 AudioJack2_Ground_Switch, J7 DIN-5, J8 AudioJack2_Ground_Switch, J9 AudioJack2_Ground_Switch, Q1 MMBT2222A, Q2 MMBT2222A, SW1 Rotary_Encoder_Switch, U1 TL072, U2 EL814, U3 MCP4728

Commit message: Replace PJ301 w PJ321
Parts:
- J10, J11, J12, J13, J3, J5, J6, J8, J9: footprint Connector_Audio:Jack_3.5mm_QingPu_WQP-PJ398SM_Vertical_CircularHoles -> Connector_Audio:AudioJack3StereoNarrow-PJ-321
Changed lines of the file:
@@
 F 0 "J5" H 9367 2971 50  0000 R CNN
 F 1 "AudioJack2_Ground_Switch" H 9367 2880 50  0000 R CNN
-F 2 "Connector_Audio:Jack_3.5mm_QingPu_WQP-PJ398SM_Vertical_CircularHoles" H 9600 2900 50  0001 C CNN
+F 2 "Connector_Audio:AudioJack3StereoNarrow-PJ-321" H 9600 2900 50  0001 C CNN
 F 3 "~" H 9600 2900 50  0001 C CNN
 F 4 "CV1 Out" H 9600 2900 50  0001 C CNN "Function"
@@
 F 0 "J6" H 9367 3421 50  0000 R CNN
 F 1 "AudioJack2_Ground_Switch" H 9367 3330 50  0000 R CNN
-F 2 "Connector_Audio:Jack_3.5mm_QingPu_WQP-PJ398SM_Vertical_CircularHoles" H 9600 3350 50  0001 C CNN
+F 2 "Connector_Audio:AudioJack3StereoNarrow-PJ-321" H 9600 3350 50  0001 C CNN
 F 3 "~" H 9600 3350 50  0001 C CNN
 F 4 "CV2 out" H 9600 3350 50  0001 C CNN "Function"
@@
 F 0 "J8" H 9367 3871 50  0000 R CNN
 F 1 "AudioJack2_Ground_Switch" H 9367 3780 50  0000 R CNN
-F 2 "Connector_Audio:Jack_3.5mm_QingPu_WQP-PJ398SM_Vertical_CircularHoles" H 9600 3800 50  0001 C CNN
+F 2 "Connector_Audio:AudioJack3StereoNarrow-PJ-321" H 9600 3800 50  0001 C CNN
 F 3 "~" H 9600 3800 50  0001 C CNN
 	1    9600 3800
@@
 F 0 "J9" H 9367 4271 50  0000 R CNN
 F 1 "AudioJack2_Ground_Switch" H 9367 4180 50  0000 R CNN
-F 2 "Connector_Audio:Jack_3.5mm_QingPu_WQP-PJ398SM_Vertical_CircularHoles" H 9600 4200 50  0001 C CNN
+F 2 "Connector_Audio:AudioJack3StereoNarrow-PJ-321" H 9600 4200 50  0001 C CNN
 F 3 "~" H 9600 4200 50  0001 C CNN
 	1    9600 4200
@@
 F 0 "J10" H 9367 4721 50  0000 R CNN
 F 1 "AudioJack2_Ground_Switch" H 9367 4630 50  0000 R CNN
-F 2 "Connector_Audio:Jack_3.5mm_QingPu_WQP-PJ398SM_Vertical_CircularHoles" H 9600 4650 50  0001 C CNN
+F 2 "Connector_Audio:AudioJack3StereoNarrow-PJ-321" H 9600 4650 50  0001 C CNN
 F 3 "~" H 9600 4650 50  0001 C CNN
 	1    9600 4650
@@
 F 0 "J11" H 9367 5171 50  0000 R CNN
 F 1 "AudioJack2_Ground_Switch" H 9367 5080 50  0000 R CNN
-F 2 "Connector_Audio:Jack_3.5mm_QingPu_WQP-PJ398SM_Vertical_CircularHoles" H 9600 5100 50  0001 C CNN
+F 2 "Connector_Audio:AudioJack3StereoNarrow-PJ-321" H 9600 5100 50  0001 C CNN
 F 3 "~" H 9600 5100 50  0001 C CNN
 	1    9600 5100
@@
 F 0 "J12" H 9367 5621 50  0000 R CNN
 F 1 "AudioJack2_Ground_Switch" H 9367 5530 50  0000 R CNN
-F 2 "Connector_Audio:Jack_3.5mm_QingPu_WQP-PJ398SM_Vertical_CircularHoles" H 9600 5550 50  0001 C CNN
+F 2 "Connector_Audio:AudioJack3StereoNarrow-PJ-321" H 9600 5550 50  0001 C CNN
 F 3 "~" H 9600 5550 50  0001 C CNN
 	1    9600 5550
@@
 F 0 "J13" H 9367 6021 50  0000 R CNN
 F 1 "AudioJack2_Ground_Switch" H 9367 5930 50  0000 R CNN
-F 2 "Connector_Audio:Jack_3.5mm_QingPu_WQP-PJ398SM_Vertical_CircularHoles" H 9600 5950 50  0001 C CNN
+F 2 "Connector_Audio:AudioJack3StereoNarrow-PJ-321" H 9600 5950 50  0001 C CNN
 F 3 "~" H 9600 5950 50  0001 C CNN
 	1    9600 5950
@@
 F 0 "J3" H 9367 2321 50  0000 R CNN
 F 1 "AudioJack2_Ground_Switch" H 9367 2230 50  0000 R CNN
-F 2 "Connector_Audio:Jack_3.5mm_QingPu_WQP-PJ398SM_Vertical_CircularHoles" H 9600 2250 50  0001 C CNN
+F 2 "Connector_Audio:AudioJack3StereoNarrow-PJ-321" H 9600 2250 50  0001 C CNN
 F 3 "~" H 9600 2250 50  0001 C CNN
 F 4 "VC input" H 9600 2250 50  0001 C CNN "Function"

Commit message: Jack I/O
Label jacks
Voltage div on CV in / A3
Parts:
- added R10, R8: 10k, Resistor_SMD:R_0805_2012Metric_Pad1.15x1.40mm_HandSolder, symbol Device:R
- J10: value AudioJack2_Ground_Switch -> Gate1
- J11: value AudioJack2_Ground_Switch -> Gate2
- J12: value AudioJack2_Ground_Switch -> Gate3
- J13: value AudioJack2_Ground_Switch -> Gate4
- J3: value AudioJack2_Ground_Switch -> CV in
- J5: value AudioJack2_Ground_Switch -> CV1
- J6: value AudioJack2_Ground_Switch -> CV2
- J8: value AudioJack2_Ground_Switch -> CV3
- J9: value AudioJack2_Ground_Switch -> CV4
- renumbered R9 to R11, R10 to R12, R11 to R13, R12 to R14, R13 to R15, R14 to R16, R15 to R17, R16 to R18, R17 to R19, R18 to R20, R19 to R21, R20 to R22, R21 to R23, R22 to R24, R23 to R25, R24 to R26, R8 to R9
Connections:
- wire segments 247 -> 252
Changed lines of the file:
@@
 $EndComp
 $Comp
-L Device:R R16
+L Device:R R18
 U 1 1 5C1CFAFB
 P 1550 5100
-F 0 "R16" V 1343 5100 50  0000 C CNN
+F 0 "R18" V 1343 5100 50  0000 C CNN
 F 1 "680R" V 1434 5100 50  0000 C CNN
 F 2 "Resistor_SMD:R_0805_2012Metric_Pad1.15x1.40mm_HandSolder" V 1480 5100 50  0001 C CNN
@@
 $EndComp
 $Comp
-L Device:R R17
+L Device:R R19
 U 1 1 5C1CFC0E
 P 1550 5400
-F 0 "R17" V 1343 5400 50  0000 C CNN
+F 0 "R19" V 1343 5400 50  0000 C CNN
 F 1 "680R" V 1434 5400 50  0000 C CNN
 F 2 "Resistor_SMD:R_0805_2012Metric_Pad1.15x1.40mm_HandSolder" V 1480 5400 50  0001 C CNN
@@
 $EndComp
 $Comp
-L Device:R R18
+L Device:R R20
 U 1 1 5C1CFC52
 P 1550 5750
-F 0 "R18" V 1343 5750 50  0000 C CNN
+F 0 "R20" V 1343 5750 50  0000 C CNN
 F 1 "680R" V 1434 5750 50  0000 C CNN
 F 2 "Resistor_SMD:R_0805_2012Metric_Pad1.15x1.40mm_HandSolder" V 1480 5750 50  0001 C CNN
@@
 $EndComp
 $Comp
-L Device:R R19
+L Device:R R21
 U 1 1 5C1CFCA2
 P 1550 6050
-F 0 "R19" V 1343 6050 50  0000 C CNN
+F 0 "R21" V 1343 6050 50  0000 C CNN
 F 1 "680R" V 1434 6050 50  0000 C CNN
 F 2 "Resistor_SMD:R_0805_2012Metric_Pad1.15x1.40mm_HandSolder" V 1480 6050 50  0001 C CNN
@@
 $EndComp
 $Comp
-L Device:R R12
+L Device:R R14
 U 1 1 5C1CFCF0
 P 1500 3650
-F 0 "R12" V 1293 3650 50  0000 C CNN
+F 0 "R14" V 1293 3650 50  0000 C CNN
 F 1 "220R" V 1384 3650 50  0000 C CNN
 F 2 "Resistor_SMD:R_0805_2012Metric_Pad1.15x1.40mm_HandSolder" V 1430 3650 50  0001 C CNN
@@
 Connection ~ 750  6050
 $Comp
-L Device:R R11
+L Device:R R13
 U 1 1 5C1DFF32
 P 2850 3400
-F 0 "R11" H 2780 3354 50  0000 R CNN
+F 0 "R13" H 2780 3354 50  0000 R CNN
 F 1 "1k" H 2780 3445 50  0000 R CNN
 F 2 "Resistor_SMD:R_0805_2012Metric_Pad1.15x1.40mm_HandSolder" V 2780 3400 50  0001 C CNN
@@
 $EndComp
 $Comp
-L Device:R R13
+L Device:R R15
 U 1 1 5C1E3615
 P 2500 4100
-F 0 "R13" H 2430 4054 50  0000 R CNN
+F 0 "R15" H 2430 4054 50  0000 R CNN
 F 1 "1k" H 2430 4145 50  0000 R CNN
 F 2 "Resistor_SMD:R_0805_2012Metric_Pad1.15x1.40mm_HandSolder" V 2430 4100 50  0001 C CNN
@@
 	2500 3850 2650 3850
 $Comp
-L Device:R R9
+L Device:R R11
 U 1 1 5C1E9F2A
 P 6100 2800
-F 0 "R9" H 6250 2900 50  0000 R CNN
+F 0 "R11" H 6250 2900 50  0000 R CNN
 F 1 "8k2" H 6300 2800 50  0000 R CNN
 F 2 "Resistor_SMD:R_0805_2012Metric_Pad1.15x1.40mm_HandSolder" V 6030 2800 50  0001 C CNN
@@
 $EndComp
 $Comp
-L Device:R R10
+L Device:R R12
 U 1 1 5C1E9FAC
 P 6200 2800
-F 0 "R10" H 6100 2900 50  0000 R CNN
+F 0 "R12" H 6100 2900 50  0000 R CNN
 F 1 "8k2" H 6100 2800 50  0000 R CNN
 F 2 "Resistor_SMD:R_0805_2012Metric_Pad1.15x1.40mm_HandSolder" V 6130 2800 50  0001 C CNN
@@
 $EndComp
 $Comp
-L Device:R R23
+L Device:R R25
 U 1 1 5C26F86C
 P 3650 7050
-F 0 "R23" V 3443 7050 50  0000 C CNN
+F 0 "R25" V 3443 7050 50  0000 C CNN
 F 1 "10k" V 3534 7050 50  0000 C CNN
 F 2 "Resistor_SMD:R_0805_2012Metric_Pad1.15x1.40mm_HandSolder" V 3580 7050 50  0001 C CNN
@@
 $EndComp
 $Comp
-L Device:R R24
+L Device:R R26
 U 1 1 5C26F900
 P 3650 7250
-F 0 "R24" V 3443 7250 50  0000 C CNN
+F 0 "R26" V 3443 7250 50  0000 C CNN
 F 1 "10k" V 3534 7250 50  0000 C CNN
 F 2 "Resistor_SMD:R_0805_2012Metric_Pad1.15x1.40mm_HandSolder" V 3580 7250 50  0001 C CNN
@@
 P 9600 2900
 F 0 "J5" H 9367 2971 50  0000 R CNN
-F 1 "AudioJack2_Ground_Switch" H 9367 2880 50  0000 R CNN
+F 1 "CV1" H 9367 2880 50  0000 R CNN
 F 2 "Connector_Audio:AudioJack3StereoNarrow-PJ-321" H 9600 2900 50  0001 C CNN
 F 3 "~" H 9600 2900 50  0001 C CNN
@@
 P 9600 3350
 F 0 "J6" H 9367 3421 50  0000 R CNN
-F 1 "AudioJack2_Ground_Switch" H 9367 3330 50  0000 R CNN
+F 1 "CV2" H 9367 3330 50  0000 R CNN
 F 2 "Connector_Audio:AudioJack3StereoNarrow-PJ-321" H 9600 3350 50  0001 C CNN
 F 3 "~" H 9600 3350 50  0001 C CNN
@@
 $EndComp
 $Comp
-L Device:R R20
+L Device:R R22
 U 1 1 5C30AA3A
 P 1550 6350
-F 0 "R20" V 1343 6350 50  0000 C CNN
+F 0 "R22" V 1343 6350 50  0000 C CNN
 F 1 "680R" V 1434 6350 50  0000 C CNN
 F 2 "Resistor_SMD:R_0805_2012Metric_Pad1.15x1.40mm_HandSolder" V 1480 6350 50  0001 C CNN
@@
 SDA
 $Comp
-L Device:R R22
+L Device:R R24
 U 1 1 5C3D162F
 P 1700 7050
-F 0 "R22" V 1493 7050 50  0000 C CNN
+F 0 "R24" V 1493 7050 50  0000 C CNN
 F 1 "10k" V 1584 7050 50  0000 C CNN
 F 2 "Resistor_SMD:R_0805_2012Metric_Pad1.15x1.40mm_HandSolder" V 1630 7050 50  0001 C CNN
@@
 $EndComp
 $Comp
-L Device:R R21
+L Device:R R23
 U 1 1 5C41F476
 P 1550 6600
-F 0 "R21" V 1343 6600 50  0000 C CNN
+F 0 "R23" V 1343 6600 50  0000 C CNN
 F 1 "680R" V 1434 6600 50  0000 C CNN
 F 2 "Resistor_SMD:R_0805_2012Metric_Pad1.15x1.40mm_HandSolder" V 1480 6600 50  0001 C CNN
@@
 Wire Wire Line
 	5350 4500 5050 4500
-Text GLabel 9000 2250 0    50   Input ~ 0
+Text GLabel 8550 2250 0    50   Input ~ 0
 A3
 Text GLabel 9100 5550 0    50   Input ~ 0
@@
 P 9600 3800
 F 0 "J8" H 9367 3871 50  0000 R CNN
-F 1 "AudioJack2_Ground_Switch" H 9367 3780 50  0000 R CNN
+F 1 "CV3" H 9367 3780 50  0000 R CNN
 F 2 "Connector_Audio:AudioJack3StereoNarrow-PJ-321" H 9600 3800 50  0001 C CNN
 F 3 "~" H 9600 3800 50  0001 C CNN
@@
 P 9600 4200
 F 0 "J9" H 9367 4271 50  0000 R CNN
-F 1 "AudioJack2_Ground_Switch" H 9367 4180 50  0000 R CNN
+F 1 "CV4" H 9367 4180 50  0000 R CNN
 F 2 "Connector_Audio:AudioJack3StereoNarrow-PJ-321" H 9600 4200 50  0001 C CNN
 F 3 "~" H 9600 4200 50  0001 C CNN
@@
 P 9600 4650
 F 0 "J10" H 9367 4721 50  0000 R CNN
-F 1 "AudioJack2_Ground_Switch" H 9367 4630 50  0000 R CNN
+F 1 "Gate1" H 9367 4630 50  0000 R CNN
 F 2 "Connector_Audio:AudioJack3StereoNarrow-PJ-321" H 9600 4650 50  0001 C CNN
 F 3 "~" H 9600 4650 50  0001 C CNN
@@
 P 9600 5100
 F 0 "J11" H 9367 5171 50  0000 R CNN
-F 1 "AudioJack2_Ground_Switch" H 9367 5080 50  0000 R CNN
+F 1 "Gate2" H 9367 5080 50  0000 R CNN
 F 2 "Connector_Audio:AudioJack3StereoNarrow-PJ-321" H 9600 5100 50  0001 C CNN
 F 3 "~" H 9600 5100 50  0001 C CNN
@@
 P 9600 5550
 F 0 "J12" H 9367 5621 50  0000 R CNN
-F 1 "AudioJack2_Ground_Switch" H 9367 5530 50  0000 R CNN
+F 1 "Gate3" H 9367 5530 50  0000 R CNN
 F 2 "Connector_Audio:AudioJack3StereoNarrow-PJ-321" H 9600 5550 50  0001 C CNN
 F 3 "~" H 9600 5550 50  0001 C CNN
@@
 P 9600 5950
 F 0 "J13" H 9367 6021 50  0000 R CNN
-F 1 "AudioJack2_Ground_Switch" H 9367 5930 50  0000 R CNN
+F 1 "Gate4" H 9367 5930 50  0000 R CNN
 F 2 "Connector_Audio:AudioJack3StereoNarrow-PJ-321" H 9600 5950 50  0001 C CNN
 F 3 "~" H 9600 5950 50  0001 C CNN
@@
 P 9600 2250
 F 0 "J3" H 9367 2321 50  0000 R CNN
-F 1 "AudioJack2_Ground_Switch" H 9367 2230 50  0000 R CNN
+F 1 "CV in" H 9367 2230 50  0000 R CNN
 F 2 "Connector_Audio:AudioJack3StereoNarrow-PJ-321" H 9600 2250 50  0001 C CNN
 F 3 "~" H 9600 2250 50  0001 C CNN
@@
 	-1   0    0    -1
 $EndComp
-Wire Wire Line
-	9000 2250 9400 2250
 Wire Wire Line
 	9400 2150 9250 2150
@@
 I2C DAC
 $Comp
-L Device:R R14
+L Device:R R16
 U 1 1 5C717B18
 P 7700 4250
-F 0 "R14" H 7630 4204 50  0000 R CNN
+F 0 "R16" H 7630 4204 50  0000 R CNN
 F 1 "0R" H 7630 4295 50  0000 R CNN
 F 2 "Resistor_SMD:R_0805_2012Metric_Pad1.15x1.40mm_HandSolder" V 7630 4250 50  0001 C CNN
@@
 $EndComp
 $Comp
-L Device:R R15
+L Device:R R17
 U 1 1 5C717C4A
 P 7600 4850
-F 0 "R15" H 7530 4804 50  0000 R CNN
+F 0 "R17" H 7530 4804 50  0000 R CNN
 F 1 "0R" H 7530 4895 50  0000 R CNN
 F 2 "Resistor_SMD:R_0805_2012Metric_Pad1.15x1.40mm_HandSolder" V 7530 4850 50  0001 C CNN
@@
 $EndComp
 $Comp
-L Device:R R8
+L Device:R R9
 U 1 1 5C800F7E
 P 2500 2450
-F 0 "R8" H 2430 2404 50  0000 R CNN
+F 0 "R9" H 2430 2404 50  0000 R CNN
 F 1 "1k" H 2430 2495 50  0000 R CNN
 F 2 "Resistor_SMD:R_0805_2012Metric_Pad1.15x1.40mm_HandSolder" V 2430 2450 50  0001 C CNN
@@
 	4550 5200 4600 5200
 $Comp
-L power:GND #PWR0101
+L power:GND #PWR015
 U 1 1 5C912A2F
 P 4600 5300
-F 0 "#PWR0101" H 4600 5050 50  0001 C CNN
+F 0 "#PWR015" H 4600 5050 50  0001 C CNN
 F 1 "GND" H 4605 5127 50  0000 C CNN
 F 2 "" H 4600 5300 50  0001 C CNN
@@
 Wire Wire Line
 	4600 5200 4650 5200
+$Comp
+L Device:R R8
+U 1 1 5C272108
+P 9000 2250
+F 0 "R8" V 8793 2250 50  0000 C CNN
+F 1 "10k" V 8884 2250 50  0000 C CNN
+F 2 "Resistor_SMD:R_0805_2012Metric_Pad1.15x1.40mm_HandSolder" V 8930 2250 50  0001 C CNN
+F 3 "~" H 9000 2250 50  0001 C CNN
+	1    9000 2250
+	0    1    1    0
+$EndComp
+$Comp
+L Device:R R10
+U 1 1 5C27224E
+P 8800 2450
+F 0 "R10" H 8700 2550 50  0000 R CNN
+F 1 "10k" H 8700 2450 50  0000 R CNN
+F 2 "Resistor_SMD:R_0805_2012Metric_Pad1.15x1.40mm_HandSolder" V 8730 2450 50  0001 C CNN
+F 3 "~" H 8800 2450 50  0001 C CNN
+	1    8800 2450
+	-1   0    0    1
+$EndComp
+Wire Wire Line
+	8550 2250 8800 2250
+Wire Wire Line
+	9150 2250 9400 2250
+Wire Wire Line
+	8800 2300 8800 2250
+Connection ~ 8800 2250
+Wire Wire Line
+	8800 2250 8850 2250
+Wire Wire Line
+	8800 2600 8800 2800
+Wire Wire Line
+	8800 2800 9250 2800
 $EndSCHEMATC

Commit message: Fixed Analog voltage
Encoder module replace
PCB reorganize
Added Analogue supply - not done
changed Jacks
etc
Parts:
- removed R25, R26: 10k, Resistor_SMD:R_0805_2012Metric_Pad1.15x1.40mm_HandSolder, symbol Device:R
- removed SW1: Rotary_Encoder_Switch, Rotary_Encoder:RotaryEncoder_Alps_EC11E-Switch_Vertical_H20mm, symbol Device:Rotary_Encoder_Switch
- added C? (x2): 100uF 16v, Capacitor_THT:CP_Radial_D5.0mm_P2.50mm, symbol Device:CP
- added C? (x2): 100n, Capacitor_SMD:C_0805_2012Metric_Pad1.15x1.40mm_HandSolder, symbol Device:C
- added SW1: KY40_Rotary_Encoder_Module, Rotary_Encoder:KY-40-rotary-encoder-board, symbol Module:KY40_Rotary_Encoder_Module
- added U?: TL072, Package_SO:SO-8_5.3x6.2mm_P1.27mm, symbol Amplifier_Operational:TL072
- C1: value CP -> 100uF
- C2, C3: value C -> 100n
- D1: value LED -> LED1
- D2: value LED -> LED2
- D3: value LED -> LED3
- D4: value LED -> LED4
- D5: value LED -> LEDset1
- D6: value LED -> LEDset2
- J1: value Barrel_Jack -> Vin 7-12v
- J10, J11, J12, J13, J3, J5, J6, J8, J9: symbol Connector:AudioJack2_Ground_Switch -> Connector:AudioJack2
- J2: value DIN-5 -> MIDI OUT
- J7: value DIN-5 -> MIDI IN
Connections:
- wire segments 252 -> 239
Other:
- moved on the sheet: C5, C6, C7, R24

Commit message: Board interconnectors
Gate and I2C signals prepared
Parts:
- added J1: Doepfer connector, Connector_PinSocket_2.54mm:PinSocket_2x08_P2.54mm_Vertical, symbol Connector_Generic:Conn_02x08_Counter_Clockwise
- added J12: A6 A7, Connector_PinSocket_2.54mm:PinSocket_1x03_P2.54mm_Vertical, symbol Connector:Conn_01x03_Male
- added J16, J17: Conn_01x06_Male, Connector_PinSocket_2.54mm:PinSocket_1x06_P2.54mm_Vertical, symbol Connector:Conn_01x06_Male
- gave numbers to parts that had none: 5
- renumbered C6 to C10, C7 to C11, C4 to C8, C5 to C9, J9 to J10, J10 to J11, J11 to J13, J12 to J14, J13 to J15, J1 to J2, J2 to J3, J3 to J4, J4 to J5, J5 to J6, J6 to J7, J7 to J8, J8 to J9
Connections:
- wire segments 239 -> 305
Other:
- note added: "Board intercon"
- note added: "MIDI OUT"
- note added: "POWER"
- moved on the sheet: C1, C2, C3, C4, C5, C6, C7, J2, R1, R3, R4, RV1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

Commit message: Analogue card routed - no GND
Parts:
- removed J12: A6 A7, Connector_PinSocket_2.54mm:PinSocket_1x03_P2.54mm_Vertical, symbol Connector:Conn_01x03_Male
- added J12, J18: GateConn, Connector_PinSocket_2.54mm:PinSocket_1x06_P2.54mm_Vertical, symbol Connector:Conn_01x06_Male
- C8: value C -> 100n
- J1: symbol Connector_Generic:Conn_02x08_Counter_Clockwise -> Connector_Generic:Conn_02x08_Odd_Even
- J16, J17: value Conn_01x06_Male -> I2C_Conn
- J5: value Conn_01x04 -> Power Conn
Connections:
- net labels added: -12v, 12v, A6, A7, Vout1, Vout2
- wire segments 305 -> 321
Other:
- moved on the sheet: C10, C11, C9, R24, SW1

Commit message: AJ_SO8 pad for Op Amp
Parts:
- added J19: CV7 in, Connector_Audio:AudioJack3StereoNarrow-PJ-321, symbol Connector:AudioJack2
- added J20: CV3 in, Connector_Audio:AudioJack3StereoNarrow-PJ-321, symbol Connector:AudioJack2
- added R25, R26, R27, R28: 10k, Resistor_SMD:R_0805_2012Metric_Pad1.15x1.40mm_HandSolder, symbol Device:R
- J4: value CV in -> CV6 in
- U1: footprint Package_SO:SO-8_5.3x6.2mm_P1.27mm -> AJ-Dropbox-Kicad:AJ_SO-8_5.3x6.2mm_P1.27mm
Connections:
- wire segments 321 -> 340
Other:
- moved on the sheet: J10, J11, J13, J14, J15, J4, J6, J7, J9, R10, R2, R4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
