File: _saved_Kicad-Midi2CV.sch (KiCad schematic (older format))
At the start: 25 parts, among them IC1 MCP4725module, IC2 MCP4725module, J1 Barrel_Jack, J2 Conn_01x04, J3 DIN-5, Q1 MMBT2222A, SW1 Rotary_Encoder_Switch, U1 MCP4728, U2 EL814

Commit message: Footprints
footprint PL814
Parts:
- J2: footprint (none) -> Connector_PinHeader_2.54mm:PinHeader_1x04_P2.54mm_Vertical
- U1: renamed from U2; footprint OptoDevice:Panasonic_APV-AQY_SSOP-4_4.45x2.65mm_P1.27mm -> Package_DIP:DIP-4_W7.62mm_LongPads
- renumbered U1 to U2
Connections:
- wire segments 115 -> 117
Changed lines of the file:
@@
 $EndComp
 $Comp
-L Isolator:EL814 U2
+L Isolator:EL814 U1
 U 1 1 5C1C075E
 P 2250 2500
-F 0 "U2" H 2250 2825 50  0000 C CNN
+F 0 "U1" H 2250 2825 50  0000 C CNN
 F 1 "EL814" H 2250 2734 50  0000 C CNN
-F 2 "OptoDevice:Panasonic_APV-AQY_SSOP-4_4.45x2.65mm_P1.27mm" H 2050 2300 50  0001 L CIN
+F 2 "Package_DIP:DIP-4_W7.62mm_LongPads" H 2050 2300 50  0001 L CIN
 F 3 "http://www.everlight.com/file/ProductFile/EL814.pdf" H 2275 2500 50  0001 L CNN
 	1    2250 2500
@@
 $EndComp
 $Comp
-L Analog_DAC:MCP4728 U1
+L Analog_DAC:MCP4728 U2
 U 1 1 5C1C0F59
 P 7200 4800
-F 0 "U1" H 7200 5278 50  0000 C CNN
+F 0 "U2" H 7200 5278 50  0000 C CNN
 F 1 "MCP4728" H 7200 5187 50  0000 C CNN
 F 2 "Package_SO:MSOP-10_3x3mm_P0.5mm" H 7200 4200 50  0001 C CNN
@@
 F 0 "J2" H 6080 1792 50  0000 L CNN
 F 1 "Conn_01x04" H 6080 1701 50  0000 L CNN
-F 2 "" H 6000 1800 50  0001 C CNN
+F 2 "Connector_PinHeader_2.54mm:PinHeader_1x04_P2.54mm_Vertical" H 6000 1800 50  0001 C CNN
 F 3 "~" H 6000 1800 50  0001 C CNN
 	1    6000 1800
@@
 Wire Wire Line
 	3500 5400 4300 5400
+Wire Wire Line
+	2500 950  5000 950
+Wire Wire Line
+	5000 950  5000 1600
+Connection ~ 2500 950
+Connection ~ 5000 1600
 $EndSCHEMATC
