File: _autosave-Kicad-Midi2CV.kicad_pcb (KiCad board)
At the start: 2 copper layers, 99.7 x 99.7 mm, 78 parts, among them IC1 MCP4725module, IC2 MCP4725module, J1 Doepfer connector, J10 CV4, J11 Gate1, J12 GateConn, J13 Gate2, J14 Gate3, J15 Gate4, J16 I2C_Conn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

Commit message: Reorganize PCB
make sure the board assembles when sandwiched
Parts:
- moved R8 94.1 mm to (40.0, 120.7)
- moved C3 55.0 mm to (48.3, 92.1)
- moved R18 49.6 mm to (117.5, 77.5)
- moved D1 49.5 mm to (122.6, 80.0)
- moved R19 38.8 mm to (117.5, 72.4)
- moved D2 38.7 mm to (122.6, 74.9)
- moved R24 36.8 mm to (114.3, 31.8)
- moved SW1 36.2 mm to (121.3, 37.5)
- moved R7 30.3 mm to (104.1, 106.0)
- moved U2 29.3 mm to (102.2, 95.9), turned to 180 degrees
- moved R20 28.6 mm to (117.5, 67.3)
- moved D3 28.6 mm to (122.6, 69.8)
- moved R14 25.1 mm to (102.9, 88.9)
- moved R6 23.9 mm to (99.7, 106.0), turned to 180 degrees
- moved C2 23.3 mm to (82.3, 106.7)
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