File: Kicad-Midi2CV.kicad_pcb (KiCad board)
At the start: 2 copper layers, 99.7 x 99.7 mm, 85 parts, among them IC1 MCP4725module, IC2 MCP4725module, J1 Doepfer connector, J10 CV4, J11 Gate1, J12 GateConn, J13 Gate2, J14 Gate3, J15 Gate4, J16 I2C_Conn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

Commit message: R and C Labels on analogue side
Parts:
- C10: value 10n -> 100n
- moved REF** 2.45 mm to (92.8, 31.8)
Changed lines of the file:
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@@
   )
   (page A4)
+  (title_block
+    (title Midi2CV)
+    (date 2019-01-21)
+    (rev "Rev B")
+    (company "Johansen Engineering")
+  )
   (layers
     (0 F.Cu signal)
@@
     (38 B.Mask user)
     (39 F.Mask user)
-    (40 Dwgs.User user hide)
+    (40 Dwgs.User user)
     (41 Cmts.User user)
     (42 Eco1.User user)
@@
   )
   (module MountingHole:MountingHole_3.2mm_M3_Pad_Via (layer F.Cu)
-    (at 95.25 31.75)
+    (at 92.8 31.75)
     (descr "Mounting Hole 3.2mm, M3")
     (tags "mounting hole 3.2mm m3")
@@
       (effects (font (size 1 1) (thickness 0.15)))
     )
-    (fp_text value 10k (at 0 1.65 180) (layer F.Fab)
+    (fp_text value 10k (at -0.512 1.65 180) (layer F.SilkS)
       (effects (font (size 1 1) (thickness 0.15)))
     )
@@
     (tags "capacitor handsolder")
     (attr smd)
-    (fp_text reference C9 (at 0 -1.65 180) (layer F.SilkS)
+    (fp_text reference C9 (at 3.581317 1.670764 180) (layer F.SilkS)
       (effects (font (size 1 1) (thickness 0.15)))
     )
-    (fp_text value 10n (at 0 1.65 180) (layer F.Fab)
+    (fp_text value 10n (at 0 1.65 180) (layer F.SilkS)
       (effects (font (size 1 1) (thickness 0.15)))
     )
@@
     (tags "capacitor handsolder")
     (attr smd)
-    (fp_text reference C10 (at 0 -1.65 180) (layer F.SilkS)
+    (fp_text reference C10 (at 3.181317 -0.589236 180) (layer F.SilkS)
       (effects (font (size 1 1) (thickness 0.15)))
     )
-    (fp_text value 10n (at 0 1.65 180) (layer F.Fab)
+    (fp_text value 100n (at 2.981317 1.410764 180) (layer F.SilkS)
       (effects (font (size 1 1) (thickness 0.15)))
     )
@@
     (tags "capacitor handsolder")
     (attr smd)
-    (fp_text reference C11 (at 0 -1.65 180) (layer F.SilkS)
+    (fp_text reference C11 (at 3.181317 -0.849236 180) (layer F.SilkS)
       (effects (font (size 1 1) (thickness 0.15)))
     )
-    (fp_text value 10n (at 0 1.65 180) (layer F.Fab)
+    (fp_text value 10n (at 3.181317 0.350764 180) (layer F.Fab)
       (effects (font (size 1 1) (thickness 0.15)))
     )
@@
       (effects (font (size 1 1) (thickness 0.15)))
     )
-    (fp_text value 10k (at -0.254 -1.524 180) (layer F.Fab)
+    (fp_text value 10k (at -0.512 -1.67 180) (layer F.SilkS)
       (effects (font (size 1 1) (thickness 0.15)))
     )
@@
       (effects (font (size 1 1) (thickness 0.15)))
     )
-    (fp_text value 10k (at 0 1.65 180) (layer F.Fab)
+    (fp_text value 10k (at 0 1.65 180) (layer F.SilkS)
       (effects (font (size 1 1) (thickness 0.15)))
     )
@@
     (tags "resistor handsolder")
     (attr smd)
-    (fp_text reference R28 (at 0 -1.65 180) (layer F.SilkS)
+    (fp_text reference R28 (at 3.142 -0.23 180) (layer F.SilkS)
       (effects (font (size 1 1) (thickness 0.15)))
     )
-    (fp_text value 10k (at 0 1.65 180) (layer F.Fab)
+    (fp_text value 10k (at 0.142 -1.63 180) (layer F.SilkS)
       (effects (font (size 1 1) (thickness 0.15)))
     )
@@
     (effects (font (size 1.5 1.5) (thickness 0.3)) (justify left))
   )
-  (gr_line (start 92.71 25.4) (end 92.71 125.095) (layer Dwgs.User) (width 0.15))
+  (gr_line (start 90.2 25.4) (end 90.2 125.095) (layer Dwgs.User) (width 0.15))
   (gr_line (start 25.4 75.3) (end 125.095 75.3) (layer Dwgs.User) (width 0.15))
   (gr_line (start 63.5 106.68) (end 63.5 39.37) (layer Edge.Cuts) (width 1))

Commit message: Rev B PCB - SCH - Images
Parts:
- added JP1: Tx, Connector_PinSocket_2.54mm:PinSocket_1x02_P2.54mm_Vertical, F.Cu at (76.2, 96.8)
- added JP2: Rx, Connector_PinSocket_2.54mm:PinSocket_1x02_P2.54mm_Vertical, F.Cu at (80.9, 96.8)
- C11: value 10n -> 100n
- moved R13 5.92 mm to (85.0, 97.2), turned to 0 degrees
- moved R15 3.22 mm to (90.2, 97.2), turned to 0 degrees
- moved R17 1.55 mm to (48.8, 56.2), turned to 0 degrees
Connections:
- A1 pad 1: /TX -> Net-(A1-Pad1)
- A1 pad 2: /RX -> Net-(A1-Pad2)
- Q2 pad 3: /RX -> Net-(JP2-Pad1)
- R13 pad 1: /RX -> Net-(JP2-Pad1)
Routing:
- net +5V: track 246.3 -> 188.6 mm
- net GND: track 147.6 -> 122.7 mm, vias 6 -> 8
- net /RX: track 18.0 -> 0.00 mm, vias 1 -> 0
- net Net-(A1-Pad1): track 0.00 -> 16.3 mm, vias 0 -> 1
- net Net-(A1-Pad2): track 0.00 -> 15.6 mm, vias 0 -> 1
- net Net-(JP2-Pad1): track 0.00 -> 8.89 mm
- net Net-(J4-PadT): track 18.6 -> 22.3 mm
- net /MIDI-IN: track 8.74 -> 11.4 mm
- net /Vout2: track 5.52 -> 2.93 mm
- net /TX: track 31.1 -> 31.3 mm, vias 2 -> 0
Other:
- board text added: "+5V"
- board text added: "3V3"
- board text added: "A0"
- board text added: "A1"
- board text added: "A2"
- board text added: "A5/SCL"
- board text added: "A6"
- board text added: "A7"
- board text added: "Arduino Nano USB side"
- board text added: "D10"
- board text added: "D11"
- board text added: "D12"
- board text added: "D13"
- board text added: "D2"
- board text added: "D3"
- board text added: "D4"
- board text added: "D5"
- board text added: "D9"
- board text added: "GND"
- board text added: "MIDI2CV"
- board text added: "RST"
- board text added: "RX"
- board text added: "TX"
- board text added: "Vin"
- board text added: "Vin to +5V JP"

Commit message: Minor
Other:
- board text added: "PROMESOFT Johansen Engineering MIDI2CV Rev B 2019W03"
- board text removed: "PROMESOFT Johansen Enginerring MIDI2CV Rev B 2019W3"
Changed lines of the file:
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@@
     (effects (font (size 1.5 1.5) (thickness 0.3)) (justify left mirror))
   )
-  (gr_text "PROMESOFT\nJohansen Enginerring\nMIDI2CV Rev B\n2019W3" (at 66.548 31.242) (layer F.SilkS)
-    (effects (font (size 1.5 1.5) (thickness 0.3)) (justify left))
+  (gr_text "PROMESOFT\nJohansen Engineering\nMIDI2CV Rev B\n2019W03" (at 66 32.5) (layer F.SilkS)
+    (effects (font (size 1.7 1.42) (thickness 0.3)) (justify left))
   )
   (gr_line (start 90.2 25.4) (end 90.2 125.095) (layer Dwgs.User) (width 0.15))
@@
   (segment (start 72.898 52.07) (end 67.564 52.07) (width 0.5) (layer F.Cu) (net 2))
   (segment (start 67.564 52.07) (end 66.548 53.086) (width 0.5) (layer F.Cu) (net 2))
-  (via (at 85.852 84.400001) (size 0.8) (drill 0.4) (layers F.Cu B.Cu) (net 59))
-  (segment (start 87.702001 82.55) (end 88.138 82.55) (width 0.25) (layer B.Cu) (net 59))
-  (segment (start 85.852 84.400001) (end 87.702001 82.55) (width 0.25) (layer B.Cu) (net 59))
   (segment (start 72.818764 57.070764) (end 72.898 57.15) (width 0.25) (layer F.Cu) (net 3))
   (segment (start 70.206317 57.070764) (end 72.818764 57.070764) (width 0.25) (layer F.Cu) (net 3))
@@
   (segment (start 88.138 85.09) (end 88.138 86.14) (width 0.25) (layer F.Cu) (net 58))
   (via (at 81 92.4) (size 0.8) (drill 0.4) (layers F.Cu B.Cu) (net 58))
+  (via (at 85.852 84.400001) (size 0.8) (drill 0.4) (layers F.Cu B.Cu) (net 59))
+  (segment (start 87.702001 82.55) (end 88.138 82.55) (width 0.25) (layer B.Cu) (net 59))
+  (segment (start 85.852 84.400001) (end 87.702001 82.55) (width 0.25) (layer B.Cu) (net 59))
   (segment (start 80.042856 92.28414) (end 80.042856 93.386319) (width 0.25) (layer F.Cu) (net 59))
   (segment (start 80.042856 93.386319) (end 80.892855 94.236318) (width 0.25) (layer F.Cu) (net 59))
